File: pick-to-light.kicad_pcb (KiCad board)
At the start: 4 copper layers, 38.1 x 29.8 mm, 34 parts, among them IC1 ATMEGA168PA-A, P1 CONN_02X03, P2 CONN_02X03, Q1 BC849, Q2 BC849, SW1 SW_PUSH, SW2 SW_PUSH, U1 LD1117S33TR, Y1 Crystal

Commit message: replaced chip package to QFN-32
Parts:
- C7, C8: value C -> 15pF
- IC1: footprint PTL-footprints:LQFP-32_5x5mm_Pitch0.5mm -> PTL-footprints:QFN-32-1EP_5x5mm_Pitch0.5mm
Routing:
- net Net-(IC1-Pad17): track 11.6 -> 16.9 mm, vias 0 -> 2
- net GND: track 51.9 -> 57.1 mm, vias 13 -> 15
- net RESET: track 48.5 -> 52.7 mm
- net Net-(IC1-Pad32): track 7.00 -> 8.65 mm
- net TX0: track 26.8 -> 25.3 mm
- net RX1: track 26.1 -> 26.9 mm
- net Net-(IC1-Pad2): track 7.39 -> 8.24 mm
- net A4: track 24.1 -> 25.0 mm
- net A3: track 19.1 -> 19.9 mm
- net A5: track 28.8 -> 29.7 mm
- net Net-(IC1-Pad9): track 16.9 -> 17.7 mm
- net Net-(IC1-Pad16): track 6.66 -> 7.51 mm
- net Net-(IC1-Pad15): track 33.3 -> 34.2 mm
- net Net-(IC1-Pad14): track 46.0 -> 46.8 mm
- net Net-(IC1-Pad13): track 6.63 -> 7.48 mm
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
Commit message: Sent out for prototyping
Parts:
- P1: value CONN_02X03 -> (none)
- U1: footprint TO_SOT_Packages_SMD:SOT89-3_Housing -> PTL-footprints:SOT89-3_Housing
- Y1: footprint Crystals:Crystal_HC49-U_Vertical -> PTL-footprints:Crystal_HC49-U_Vertical
- moved SW2 0.51 mm to (139.9, 91.6)
- moved Y1 0.48 mm to (109.5, 91.3)
- moved SW1 0.47 mm to (139.9, 108.5)
- moved R13 0.46 mm to (109.2, 100.7)
- moved C5 0.38 mm to (133.3, 102.6)
- moved R14 0.26 mm to (109.2, 98.6)
- moved R15 0.25 mm to (138.2, 111.1)
- moved C4 0.19 mm to (133.3, 112.0)
- moved C7 0.19 mm to (113.3, 94.2)
- moved C8 0.19 mm to (113.3, 89.3)
Routing:
- net Net-(IC1-Pad15): track 34.2 -> 39.7 mm
- net VCC: track 39.8 -> 44.1 mm
- net GND: track 57.1 -> 61.1 mm
- net RX1: track 26.9 -> 28.7 mm
- net A4: track 25.0 -> 26.6 mm
- net Net-(R4-Pad1): track 31.4 -> 30.2 mm
- net TX0: track 25.3 -> 26.3 mm
- net A5: track 29.7 -> 30.3 mm
- net Net-(IC1-Pad14): track 46.8 -> 47.4 mm
